File: Cryon-ICE/eMMC_SD.kicad_sch (KiCad schematic)
At the start: 16 parts, among them J702 MSD-7-A

Commit message: Added eMMC
Parts:
- added C704, C705, C706, C707, C708, C709, C710, C711, C712, C713: 100nF, Capacitor_SMD:C_0402_1005Metric, symbol Device:C
- added C714, C717: 4.7uF, Capacitor_SMD:C_0201_0603Metric, symbol Device:C
- added Q701: DMG1012T, Cryon_Library:DMG1012-SOT-523, symbol Transistor_FET:DMG1012T
- added R707, R708: 10k, Resistor_SMD:R_0402_1005Metric, symbol Device:R_Small_US
- added R709, R710, R711, R712, R713, R714, R715, R716, R717, R718: 49.9k, Resistor_SMD:R_0402_1005Metric, symbol Device:R_Small_US
- added R719: 0R, Resistor_SMD:R_0402_1005Metric, symbol Device:R_Small_US
- added R720: 10K, Resistor_SMD:R_0402_1005Metric, symbol Device:R_Small_US
- added U701: MX52LM08A11XVI, Cryon_Library:153BGA_11p5x13x1_MAC, symbol Cryon_Library:MX52LM08A11XVI
Connections:
- net 3V3_SD_CS: now also Q701.3 (D), R708.2
- net GND: now also J702.SW_A2, C704.1, C705.1, C706.1, C707.1, C708.1, C709.1, C710.1, C711.1, C712.1, C713.1, C714.1, C717.1, R720.2, U701.A6 (VSS), U701.C4 (VSSQ), U701.E7 (VSS), U701.G5 (VSS), U701.H10 (VSS), U701.J5 (VSS), U701.K8 (VSS), U701.N2 (VSSQ), U701.N5 (VSSQ), U701.P4 (VSSQ), U701.P6 (VSSQ)
- net SD_DET: no longer J702.SW_A2
- net VCC_3V3: now also C705.2, C706.2, C707.2, C708.2, C717.2, U701.E6 (VCC), U701.F5 (VCC), U701.J10 (VCC), U701.K9 (VCC)
- new net: C704.2, U701.C2 (VDDI)
- new net: R719.1, U701.M6 (CLK)
- new net EMMC_CLK: R719.2
- new net EMMC_CMD: R718.2, U701.M5 (CMD)
- new net EMMC_DATA0: R716.2, U701.A3 (DAT0)
- new net EMMC_DATA1: R715.2, U701.A4 (DAT1)
- new net EMMC_DATA2: R714.2, U701.A5 (DAT2)
- new net EMMC_DATA3: R713.2, U701.B2 (DAT3)
- new net EMMC_DATA4: R712.2, U701.B3 (DAT4)
- new net EMMC_DATA5: R711.2, U701.B4 (DAT5)
- new net EMMC_DATA6: R710.2, U701.B5 (DAT6)
- new net EMMC_DATA7: R709.2, U701.B6 (DAT7)
- new net EMMC_DQ: R720.1, U701.H5 (Data_Strobe)
- new net EMMC_RSTn: R717.2, U701.K5 (RST_N)
- new net SDCARD_CS: Q701.2 (S), R707.2
- new net SD_3V3: R708.1
- new net VCC_1V8: C709.2, C710.2, C711.2, C712.2, C713.2, C714.2, Q701.1 (G), R707.1, R709.1, R710.1, R711.1, R712.1, R713.1, R714.1, R715.1, R716.1, R717.1, R718.1, U701.C6 (VCCQ), U701.M4 (VCCQ), U701.N4 (VCCQ), U701.P3 (VCCQ), U701.P5 (VCCQ)
Other:
- note added: "SD Card : CS Signal Level Shift."
- note added: "eMMC"
- moved on the sheet: C701, C702, C703, D701, D702, D703, D704, D705, FB701, J702, R701, R702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
